File: 03-homelab-automation/_reference/ir-rf-blaster-pcb/xiao-c3-ir-rf.kicad_pcb (KiCad board)
At the start: 4 copper layers, 23 x 54 mm, 15 parts, among them M1 E07-M1101D, Q1 AO3400A

Commit message: feat(pcb): add silkscreen reference designators to both boards
Both generated boards previously exported empty silkscreen layers. Add
refdes for every part plus LED polarity marks so the boards can be hand-
assembled and inspected without cross-referencing the schematic.

flow-tap: J1/U1/J2/C1/J3 in a clean row above the pad field.

ir-blaster (xiao-c3-ir-rf): D1-D3 (with a cathode bar on the pin-1/west
side of each LED), R1-R5, C1-C4, Q1, A1 (XIAO), and M1 mirrored on
B.SilkS above the E07 header (the module mounts on the back).

Regenerated boards, gerbers, and top/bottom renders. DRC 0 violations /
0 unconnected on both.

Co-Authored-By: Claude Opus 4.8 <noreply@anthropic.com>
Claude-Session: https://claude.ai/code/session_01NfkRErMrPyNuft1RbpzMet
Other:
- board text added: "A1"
- board text added: "C1"
- board text added: "C2"
- board text added: "C3"
- board text added: "C4"
- board text added: "D1"
- board text added: "D2"
- board text added: "D3"
- board text added: "M1"
- board text added: "Q1"
- board text added: "R1"
- board text added: "R2"
- board text added: "R3"
- board text added: "R4"
- board text added: "R5"
