File: 03-homelab-automation/_reference/ir-rf-blaster-pcb/xiao-c3-ir-rf.kicad_pcb (KiCad board)
At the start: 4 copper layers, 23 x 54 mm, 15 parts, among them M1 E07-M1101D, Q1 AO3400A

Commit message: feat(pcb): add silkscreen reference designators to both boards (#62)
* feat(pcb): add silkscreen reference designators to both boards

Both generated boards previously exported empty silkscreen layers. Add
refdes for every part plus LED polarity marks so the boards can be hand-
assembled and inspected without cross-referencing the schematic.

flow-tap: J1/U1/J2/C1/J3 in a clean row above the pad field.

ir-blaster (xiao-c3-ir-rf): D1-D3 (with a cathode bar on the pin-1/west
side of each LED), R1-R5, C1-C4, Q1, A1 (XIAO), and M1 mirrored on
B.SilkS above the E07 header (the module mounts on the back).

Regenerated boards, gerbers, and top/bottom renders. DRC 0 violations /
0 unconnected on both.

Co-Authored-By: Claude Opus 4.8 <noreply@anthropic.com>
Claude-Session: https://claude.ai/code/session_01NfkRErMrPyNuft1RbpzMet

* fix(pcb): address silkscreen critique — drop redundant LED bars, thicker silk

- ir-blaster: remove the free-floating cathode bars; LED_D5.0mm already
  renders a cathode flat on the pin-1/west side, so the bars were a
  redundant, cosmetically nonstandard second mark. Correct the misleading
  "custom fps carry no silk" comment (they're stock fps with a hidden
  Reference; their geometric silk does render).
- both: bump silk stroke to >=0.15 mm (was 0.12 mm) to clear the common
  JLCPCB minimum so thin text can't print broken.
- flow-tap: fold the silk-text extents into the auto-outline so the top
  refdes row can't be clipped if pad/courtyard bounds shrink (outline is
  now 23.1 x 21.0 mm).

Regenerated boards, gerbers, renders. DRC 0/0 on both.

Co-Authored-By: Claude Opus 4.8 <noreply@anthropic.com>
Claude-Session: https://claude.ai/code/session_01NfkRErMrPyNuft1RbpzMet

---------

Co-authored-by: Claude Opus 4.8 <noreply@anthropic.com>
Other:
- board text added: "A1"
- board text added: "C1"
- board text added: "C2"
- board text added: "C3"
- board text added: "C4"
- board text added: "D1"
- board text added: "D2"
- board text added: "D3"
- board text added: "M1"
- board text added: "Q1"
- board text added: "R1"
- board text added: "R2"
- board text added: "R3"
- board text added: "R4"
- board text added: "R5"
