File: 06-coffee-espresso/_reference/flow-tap-pcb/flow-tap.kicad_pcb (KiCad board)
At the start: 2 copper layers, 23.2 x 19.8 mm, 5 parts, among them J1 GICAR_meter, J2 to_Vivaldi, J3 to_ito, U1 74LVC1G17

Commit message: feat(pcb): add silkscreen reference designators to both boards (#62)
* feat(pcb): add silkscreen reference designators to both boards

Both generated boards previously exported empty silkscreen layers. Add
refdes for every part plus LED polarity marks so the boards can be hand-
assembled and inspected without cross-referencing the schematic.

flow-tap: J1/U1/J2/C1/J3 in a clean row above the pad field.

ir-blaster (xiao-c3-ir-rf): D1-D3 (with a cathode bar on the pin-1/west
side of each LED), R1-R5, C1-C4, Q1, A1 (XIAO), and M1 mirrored on
B.SilkS above the E07 header (the module mounts on the back).

Regenerated boards, gerbers, and top/bottom renders. DRC 0 violations /
0 unconnected on both.

Co-Authored-By: Claude Opus 4.8 <noreply@anthropic.com>
Claude-Session: https://claude.ai/code/session_01NfkRErMrPyNuft1RbpzMet

* fix(pcb): address silkscreen critique — drop redundant LED bars, thicker silk

- ir-blaster: remove the free-floating cathode bars; LED_D5.0mm already
  renders a cathode flat on the pin-1/west side, so the bars were a
  redundant, cosmetically nonstandard second mark. Correct the misleading
  "custom fps carry no silk" comment (they're stock fps with a hidden
  Reference; their geometric silk does render).
- both: bump silk stroke to >=0.15 mm (was 0.12 mm) to clear the common
  JLCPCB minimum so thin text can't print broken.
- flow-tap: fold the silk-text extents into the auto-outline so the top
  refdes row can't be clipped if pad/courtyard bounds shrink (outline is
  now 23.1 x 21.0 mm).

Regenerated boards, gerbers, renders. DRC 0/0 on both.

Co-Authored-By: Claude Opus 4.8 <noreply@anthropic.com>
Claude-Session: https://claude.ai/code/session_01NfkRErMrPyNuft1RbpzMet

---------

Co-authored-by: Claude Opus 4.8 <noreply@anthropic.com>
Other:
- board size 23.2 x 19.8 mm -> 23.2 x 21 mm
- board text added: "C1"
- board text added: "J1"
- board text added: "J2"
- board text added: "J3"
- board text added: "U1"
Changed lines of the file:
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@@
     )
   )
-  (gr_line (start -0.05 -1.6) (end 23.1 -1.6) (layer "Edge.Cuts") (width 0.15))
-  (gr_line (start 23.1 -1.6) (end 23.1 18.15) (layer "Edge.Cuts") (width 0.15))
+  (gr_text "J1" (at 4 -0.9) (layer "F.SilkS")
+    (effects (font (size 0.8 0.8) (thickness 0.15)))
+  )
+  (gr_text "U1" (at 7 -0.9) (layer "F.SilkS")
+    (effects (font (size 0.8 0.8) (thickness 0.15)))
+  )
+  (gr_text "J2" (at 11 -0.9) (layer "F.SilkS")
+    (effects (font (size 0.8 0.8) (thickness 0.15)))
+  )
+  (gr_text "C1" (at 13 -0.9) (layer "F.SilkS")
+    (effects (font (size 0.8 0.8) (thickness 0.15)))
+  )
+  (gr_text "J3" (at 18 -0.9) (layer "F.SilkS")
+    (effects (font (size 0.8 0.8) (thickness 0.15)))
+  )
+  (gr_line (start -0.05 -2.9) (end 23.1 -2.9) (layer "Edge.Cuts") (width 0.15))
+  (gr_line (start 23.1 -2.9) (end 23.1 18.15) (layer "Edge.Cuts") (width 0.15))
   (gr_line (start 23.1 18.15) (end -0.05 18.15) (layer "Edge.Cuts") (width 0.15))
-  (gr_line (start -0.05 18.15) (end -0.05 -1.6) (layer "Edge.Cuts") (width 0.15))
+  (gr_line (start -0.05 18.15) (end -0.05 -2.9) (layer "Edge.Cuts") (width 0.15))
   (segment (start 4.0 11.5) (end 11.0 11.5) (width 0.35) (layer "F.Cu") (net 2))
   (segment (start 4.0 6.5) (end 11.0 6.5) (width 0.35) (layer "F.Cu") (net 3))
